Commit message: updated ROS and MATLAB

File: Appendix 9.4 ROS Simulation/Appendix 9.4.3 ROS Simulation Files/urdf/Robot_Arm_ASSY_half_urdf.urdf (robot description, URDF)
Before this commit: robot robot_arm_udrf, 7 links, 6 joints
Links:
- link base_link: mass 11.607 -> 47.7301508686849; geometry collision mesh filename=package://Robot_Arm_ASSY_half_urdf/meshes/base_link.STL; visual mesh filename=package://Robot_Arm_ASSY_half_urdf/meshes/base_link.STL
- link link_2: mass 0.026759 -> 0.0267586704788677; geometry collision mesh filename=package://Robot_Arm_ASSY_half_urdf/meshes/link_2.STL; visual mesh filename=package://Robot_Arm_ASSY_half_urdf/meshes/link_2.STL
- link link_3: mass 0.1963 -> 0.196297763055837; geometry collision mesh filename=package://Robot_Arm_ASSY_half_urdf/meshes/link_3.STL; visual mesh filename=package://Robot_Arm_ASSY_half_urdf/meshes/link_3.STL
- link link_4: mass 0.74143 -> 0.741427763055838; geometry collision mesh filename=package://Robot_Arm_ASSY_half_urdf/meshes/link_4.STL; visual mesh filename=package://Robot_Arm_ASSY_half_urdf/meshes/link_4.STL
- link link_5: mass 1.0591 -> 1.0590650202151; geometry collision mesh filename=package://Robot_Arm_ASSY_half_urdf/meshes/link_5.STL; visual mesh filename=package://Robot_Arm_ASSY_half_urdf/meshes/link_5.STL
- link link_6: mass 0.15645 -> 0.156447190374541; geometry collision mesh filename=package://Robot_Arm_ASSY_half_urdf/meshes/link_6.STL; visual mesh filename=package://Robot_Arm_ASSY_half_urdf/meshes/link_6.STL
- link link_7: mass 0.017016 -> 0.0170160242741333; geometry collision mesh filename=package://Robot_Arm_ASSY_half_urdf/meshes/link_7.STL; visual mesh filename=package://Robot_Arm_ASSY_half_urdf/meshes/link_7.STL
Joints:
- joint joint_1: origin xyz=0 0 0.014334 rpy=1.5708 0 0 -> xyz=0.03135 0.022079 0 rpy=1.5708 0 0
- joint joint_6: type revolute -> continuous
